File: esp32.kicad_sch (KiCad schematic)
At the start: 37 parts, among them J1 USB_C, J14 PWR_CONN, J15 SPI_0, J16 SPI_1, J3 A0, J4 A1, J5 A2, J6 D0, J7 D1, J8 USB_VOUT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

Commit message: change footprint of Vusb
Parts:
- J8: footprint Connector_PinHeader_2.54mm:PinHeader_2x01_P2.54mm_Vertical -> Connector_JST:JST_XH_B2B-XH-A_1x02_P2.50mm_Vertical
Changed lines of the file:
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@@
 			)
 		)
-		(property "Footprint" "Connector_PinHeader_2.54mm:PinHeader_2x01_P2.54mm_Vertical"
+		(property "Footprint" "Connector_JST:JST_XH_B2B-XH-A_1x02_P2.50mm_Vertical"
 			(at 27.94 48.26 0)
 			(effects

Commit message: review passed
Parts:
- removed C12: 20pF, Capacitor_SMD:C_0805_2012Metric_Pad1.18x1.45mm_HandSolder, symbol Device:C
- C18, C19: value 100n -> 100nF
- C4: value 4.7uF -> 2.2uF
- C7: value 0.1uF -> 100nF
Changed lines of the file:
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@@
 	)
 	(junction
-		(at 92.71 38.1)
-		(diameter 0)
-		(color 0 0 0 0)
-	)
-	(junction
 		(at 26.67 77.47)
 		(diameter 0)
@@
 	)
 	(junction
-		(at 92.71 30.48)
-		(diameter 0)
-		(color 0 0 0 0)
-	)
-	(junction
 		(at 102.87 30.48)
 		(diameter 0)
@@
 	(wire
 		(pts
-			(xy 92.71 38.1) (xy 96.52 38.1)
-		)
-		(stroke
-			(width 0)
-			(type default)
-		)
-	)
-	(wire
-		(pts
 			(xy 243.84 40.64) (xy 240.03 40.64)
 		)
@@
 	(wire
 		(pts
-			(xy 92.71 30.48) (xy 90.17 30.48)
-		)
-		(stroke
-			(width 0)
-			(type default)
-		)
-	)
-	(wire
-		(pts
 			(xy 246.38 39.37) (xy 243.84 39.37)
 		)
@@
 	(wire
 		(pts
-			(xy 92.71 30.48) (xy 96.52 30.48)
+			(xy 90.17 30.48) (xy 96.52 30.48)
 		)
 		(stroke
@@
 	(wire
 		(pts
-			(xy 85.09 38.1) (xy 92.71 38.1)
+			(xy 85.09 38.1) (xy 96.52 38.1)
 		)
 		(stroke
@@
 		(dnp no)
 		(property "Reference" "C18"
-			(at 17.272 80.01 0)
+			(at 16.256 80.01 0)
 			(effects
 				(font
@@
 			)
 		)
-		(property "Value" "100n"
-			(at 16.764 82.042 0)
+		(property "Value" "100nF"
+			(at 15.748 82.042 0)
 			(effects
 				(font
@@
 	)
 	(symbol
-		(lib_id "Device:C")
-		(at 92.71 34.29 0)
-		(unit 1)
-		(exclude_from_sim no)
-		(in_bom yes)
-		(on_board yes)
-		(dnp no)
-		(property "Reference" "C12"
-			(at 90.424 26.924 0)
-			(effects
-				(font
-					(size 1.27 1.27)
-				)
-				(justify left)
-			)
-		)
-		(property "Value" "20pF"
-			(at 90.17 28.702 0)
-			(effects
-				(font
-					(size 1.27 1.27)
-				)
-				(justify left)
-			)
-		)
-		(property "Footprint" "Capacitor_SMD:C_0805_2012Metric_Pad1.18x1.45mm_HandSolder"
-			(at 93.6752 38.1 0)
-			(effects
-				(font
-					(size 1.27 1.27)
-				)
-				(hide yes)
-			)
-		)
-		(property "Datasheet" "~"
-			(at 92.71 34.29 0)
-			(effects
-				(font
-					(size 1.27 1.27)
-				)
-				(hide yes)
-			)
-		)
-		(property "Description" "Unpolarized capacitor"
-			(at 92.71 34.29 0)
-			(effects
-				(font
-					(size 1.27 1.27)
-				)
-				(hide yes)
-			)
-		)
-		(pin "2"
-		)
-		(pin "1"
-		)
-		(instances
-			(project "esp32"
-				(path "/ea80ac25-815d-4e11-85a3-2f7286372b15"
-					(reference "C12")
-					(unit 1)
-				)
-			)
-		)
-	)
-	(symbol
 		(lib_id "power:PWR_FLAG")
 		(at 125.73 26.67 180)
@@
 			)
 		)
-		(property "Value" "4.7uF"
+		(property "Value" "2.2uF"
 			(at 37.338 32.766 0)
 			(effects
@@
 		(dnp no)
 		(property "Reference" "C19"
-			(at 35.56 80.01 0)
+			(at 35.56 81.534 0)
 			(effects
 				(font
@@
 			)
 		)
-		(property "Value" "100n"
-			(at 34.798 82.042 0)
+		(property "Value" "100nF"
+			(at 34.798 83.566 0)
 			(effects
 				(font
@@
 			)
 		)
-		(property "Value" "0.1uF"
+		(property "Value" "100nF"
 			(at 80.01 21.59 0)
 			(effects
